Commit message: Harden Moebius URDF for reliable Xacro parsing

File: ros2_ws/src/moebius_description/urdf/moebius_robot.urdf.xacro (robot description, xacro)
@@ -1,6 +1,6 @@
 <?xml version="1.0"?>
 <robot xmlns:xacro="http://www.ros.org/wiki/xacro" name="moebius_robot">
-  <!-- Approximate dimensions derived from the supplied robot image and legacy config.
-       Replace these properties with measured values without changing the link tree. -->
+  <!-- Parametric approximation based on the supplied robot image and legacy dimensions.
+       Measure the real chassis and edit only these properties. -->
   <xacro:property name="pi" value="3.141592653589793"/>
   <xacro:property name="wheel_radius" value="0.040"/>
@@ -15,9 +15,7 @@
   <xacro:property name="upper_height" value="0.012"/>
   <xacro:property name="plate_gap" value="0.070"/>
-  <xacro:property name="wheel_z" value="${wheel_radius}"/>
   <material name="black"><color rgba="0.035 0.035 0.045 1"/></material>
   <material name="dark_grey"><color rgba="0.12 0.12 0.14 1"/></material>
   <material name="silver"><color rgba="0.65 0.68 0.72 1"/></material>
-  <material name="roller_grey"><color rgba="0.23 0.25 0.28 1"/></material>
   <material name="sensor_black"><color rgba="0.04 0.04 0.05 1"/></material>
   <material name="blue"><color rgba="0.05 0.28 0.75 1"/></material>
@@ -31,11 +29,11 @@
     </inertial>
   </xacro:macro>
-  <xacro:macro name="cylinder_inertial" params="mass radius length axis:='y'">
+  <xacro:macro name="wheel_inertial" params="mass radius length">
     <inertial>
       <mass value="${mass}"/>
       <origin xyz="0 0 0" rpy="0 0 0"/>
-      <inertia ixx="${mass*(3*radius*radius+length*length)/12.0}" ixy="0" ixz="0"
+      <inertia ixx="${mass*(3.0*radius*radius+length*length)/12.0}" ixy="0" ixz="0"
                iyy="${0.5*mass*radius*radius}" iyz="0"
-               izz="${mass*(3*radius*radius+length*length)/12.0}"/>
+               izz="${mass*(3.0*radius*radius+length*length)/12.0}"/>
     </inertial>
   </xacro:macro>
@@ -90,5 +88,5 @@
   <xacro:standoff name="rear_left_standoff"   x="-0.095" y="0.070"/>
   <xacro:standoff name="rear_right_standoff"  x="-0.095" y="-0.070"/>
-  <xacro:macro name="mecanum_wheel" params="prefix x y side roller_sign">
+  <xacro:macro name="mecanum_wheel" params="prefix x y roller_sign">
     <link name="${prefix}_wheel_link">
       <visual>
@@ -97,45 +95,27 @@
         <material name="dark_grey"/>
       </visual>
+      <visual>
+        <origin xyz="0 0 0" rpy="${pi/2.0} ${roller_sign*0.55} 0"/>
+        <geometry><box size="${wheel_radius*1.55} ${wheel_width*1.05} 0.008"/></geometry>
+        <material name="silver"/>
+      </visual>
       <collision>
         <origin rpy="${pi/2.0} 0 0"/>
         <geometry><cylinder radius="${wheel_radius}" length="${wheel_width}"/></geometry>
       </collision>
-      <xacro:cylinder_inertial mass="0.32" radius="${wheel_radius}" length="${wheel_width}"/>
+      <xacro:wheel_inertial mass="0.32" radius="${wheel_radius}" length="${wheel_width}"/>
     </link>
     <joint name="${prefix}_wheel_joint" type="continuous">
       <parent link="base_link"/>
       <child link="${prefix}_wheel_link"/>
-      <origin xyz="${x} ${y} 0" rpy="0 0 0"/>
+      <origin xyz="${x} ${y} 0"/>
       <axis xyz="0 1 0"/>
       <dynamics damping="0.02" friction="0.02"/>
     </joint>
-    <!-- Decorative diagonal rollers for RViz. They are fixed visuals, not contact models. -->
-    <xacro:macro name="roller" params="index angle">
-      <link name="${prefix}_roller_${index}_link">
-        <visual>
-          <origin rpy="${pi/2.0} ${roller_sign*0.75} ${angle}"/>
-          <geometry><cylinder radius="0.006" length="${wheel_width*1.18}"/></geometry>
-          <material name="roller_grey"/>
-        </visual>
-      </link>
-      <joint name="${prefix}_roller_${index}_joint" type="fixed">
-        <parent link="${prefix}_wheel_link"/>
-        <child link="${prefix}_roller_${index}_link"/>
-        <origin xyz="${wheel_radius*cos(angle)} 0 ${wheel_radius*sin(angle)}"/>
-      </joint>
-    </xacro:macro>
-    <xacro:roller index="0" angle="0.0"/>
-    <xacro:roller index="1" angle="${pi/4.0}"/>
-    <xacro:roller index="2" angle="${pi/2.0}"/>
-    <xacro:roller index="3" angle="${3*pi/4.0}"/>
-    <xacro:roller index="4" angle="${pi}"/>
-    <xacro:roller index="5" angle="${5*pi/4.0}"/>
-    <xacro:roller index="6" angle="${3*pi/2.0}"/>
-    <xacro:roller index="7" angle="${7*pi/4.0}"/>
   </xacro:macro>
-  <xacro:mecanum_wheel prefix="front_left"  x="${wheelbase/2.0}"  y="${track_width/2.0}"  side="left"  roller_sign="1"/>
-  <xacro:mecanum_wheel prefix="front_right" x="${wheelbase/2.0}"  y="${-track_width/2.0}" side="right" roller_sign="-1"/>
-  <xacro:mecanum_wheel prefix="rear_left"   x="${-wheelbase/2.0}" y="${track_width/2.0}"  side="left"  roller_sign="-1"/>
-  <xacro:mecanum_wheel prefix="rear_right"  x="${-wheelbase/2.0}" y="${-track_width/2.0}" side="right" roller_sign="1"/>
+  <xacro:mecanum_wheel prefix="front_left"  x="${wheelbase/2.0}"  y="${track_width/2.0}"  roller_sign="1"/>
+  <xacro:mecanum_wheel prefix="front_right" x="${wheelbase/2.0}"  y="${-track_width/2.0}" roller_sign="-1"/>
+  <xacro:mecanum_wheel prefix="rear_left"   x="${-wheelbase/2.0}" y="${track_width/2.0}"  roller_sign="-1"/>
+  <xacro:mecanum_wheel prefix="rear_right"  x="${-wheelbase/2.0}" y="${-track_width/2.0}" roller_sign="1"/>
   <xacro:macro name="motor" params="name x y">
     <link name="${name}_motor_link">

Commit message: Consume generated dimensions in URDF

File: ros2_ws/src/moebius_description/urdf/moebius_robot.urdf.xacro (robot description, xacro)
@@ -1,11 +1,7 @@
 <?xml version="1.0"?>
 <robot xmlns:xacro="http://www.ros.org/wiki/xacro" name="moebius_robot">
-  <!-- Parametric approximation based on the supplied robot image and legacy dimensions.
-       Measure the real chassis and edit only these properties. -->
+  <xacro:include filename="$(find moebius_description)/urdf/generated/robot_specs.xacro"/>
   <xacro:property name="pi" value="3.141592653589793"/>
-  <xacro:property name="wheel_radius" value="0.040"/>
   <xacro:property name="wheel_width" value="0.036"/>
-  <xacro:property name="wheelbase" value="0.220"/>
-  <xacro:property name="track_width" value="0.260"/>
   <xacro:property name="lower_length" value="0.300"/>
   <xacro:property name="lower_width" value="0.220"/>
@@ -19,165 +15,35 @@
   <material name="silver"><color rgba="0.65 0.68 0.72 1"/></material>
   <material name="sensor_black"><color rgba="0.04 0.04 0.05 1"/></material>
-  <material name="blue"><color rgba="0.05 0.28 0.75 1"/></material>
   <xacro:macro name="box_inertial" params="mass x y z">
-    <inertial>
-      <mass value="${mass}"/>
-      <origin xyz="0 0 0" rpy="0 0 0"/>
-      <inertia ixx="${mass*(y*y+z*z)/12.0}" ixy="0" ixz="0"
-               iyy="${mass*(x*x+z*z)/12.0}" iyz="0"
-               izz="${mass*(x*x+y*y)/12.0}"/>
-    </inertial>
+    <inertial><mass value="${mass}"/><origin xyz="0 0 0"/><inertia ixx="${mass*(y*y+z*z)/12.0}" ixy="0" ixz="0" iyy="${mass*(x*x+z*z)/12.0}" iyz="0" izz="${mass*(x*x+y*y)/12.0}"/></inertial>
   </xacro:macro>
-  <xacro:macro name="wheel_inertial" params="mass radius length">
-    <inertial>
-      <mass value="${mass}"/>
-      <origin xyz="0 0 0" rpy="0 0 0"/>
-      <inertia ixx="${mass*(3.0*radius*radius+length*length)/12.0}" ixy="0" ixz="0"
-               iyy="${0.5*mass*radius*radius}" iyz="0"
-               izz="${mass*(3.0*radius*radius+length*length)/12.0}"/>
-    </inertial>
+  <xacro:macro name="wheel" params="name x y">
+    <link name="${name}_wheel_link">
+      <visual><origin rpy="${pi/2.0} 0 0"/><geometry><cylinder radius="${wheel_radius}" length="${wheel_width}"/></geometry><material name="dark_grey"/></visual>
+      <collision><origin rpy="${pi/2.0} 0 0"/><geometry><cylinder radius="${wheel_radius}" length="${wheel_width}"/></geometry></collision>
+      <inertial><mass value="0.32"/><origin xyz="0 0 0"/><inertia ixx="0.00030" ixy="0" ixz="0" iyy="0.00026" iyz="0" izz="0.00030"/></inertial>
+    </link>
+    <joint name="${name}_wheel_joint" type="continuous"><parent link="base_link"/><child link="${name}_wheel_link"/><origin xyz="${x} ${y} 0"/><axis xyz="0 1 0"/><dynamics damping="0.02" friction="0.02"/></joint>
   </xacro:macro>
   <link name="base_footprint"/>
   <link name="base_link">
-    <visual>
-      <origin xyz="0 0 ${lower_height/2.0}"/>
-      <geometry><box size="${lower_length} ${lower_width} ${lower_height}"/></geometry>
-      <material name="black"/>
-    </visual>
-    <collision>
-      <origin xyz="0 0 ${lower_height/2.0}"/>
-      <geometry><box size="${lower_length} ${lower_width} ${lower_height}"/></geometry>
-    </collision>
+    <visual><origin xyz="0 0 ${lower_height/2.0}"/><geometry><box size="${lower_length} ${lower_width} ${lower_height}"/></geometry><material name="black"/></visual>
+    <collision><origin xyz="0 0 ${lower_height/2.0}"/><geometry><box size="${lower_length} ${lower_width} ${lower_height}"/></geometry></collision>
     <xacro:box_inertial mass="3.0" x="${lower_length}" y="${lower_width}" z="${lower_height}"/>
   </link>
-  <joint name="base_footprint_joint" type="fixed">
-    <parent link="base_footprint"/>
-    <child link="base_link"/>
-    <origin xyz="0 0 ${wheel_radius}"/>
-  </joint>
-  <link name="upper_plate_link">
-    <visual>
-      <geometry><box size="${upper_length} ${upper_width} ${upper_height}"/></geometry>
-      <material name="black"/>
-    </visual>
-    <collision>
-      <geometry><box size="${upper_length} ${upper_width} ${upper_height}"/></geometry>
-    </collision>
-    <xacro:box_inertial mass="1.0" x="${upper_length}" y="${upper_width}" z="${upper_height}"/>
-  </link>
-  <joint name="upper_plate_joint" type="fixed">
-    <parent link="base_link"/>
-    <child link="upper_plate_link"/>
-    <origin xyz="0 0 ${plate_gap}"/>
-  </joint>
-  <xacro:macro name="standoff" params="name x y">
-    <link name="${name}_link">
-      <visual>
-        <geometry><cylinder radius="0.005" length="${plate_gap-upper_height}"/></geometry>
-        <material name="silver"/>
-      </visual>
-    </link>
-    <joint name="${name}_joint" type="fixed">
-      <parent link="base_link"/>
-      <child link="${name}_link"/>
-      <origin xyz="${x} ${y} ${(plate_gap-upper_height)/2.0}"/>
-    </joint>
-  </xacro:macro>
-  <xacro:standoff name="front_left_standoff"  x="0.095"  y="0.070"/>
-  <xacro:standoff name="front_right_standoff" x="0.095"  y="-0.070"/>
-  <xacro:standoff name="rear_left_standoff"   x="-0.095" y="0.070"/>
-  <xacro:standoff name="rear_right_standoff"  x="-0.095" y="-0.070"/>
-  <xacro:macro name="mecanum_wheel" params="prefix x y roller_sign">
-    <link name="${prefix}_wheel_link">
-      <visual>
-        <origin rpy="${pi/2.0} 0 0"/>
-        <geometry><cylinder radius="${wheel_radius}" length="${wheel_width}"/></geometry>
-        <material name="dark_grey"/>
-      </visual>
-      <visual>
-        <origin xyz="0 0 0" rpy="${pi/2.0} ${roller_sign*0.55} 0"/>
-        <geometry><box size="${wheel_radius*1.55} ${wheel_width*1.05} 0.008"/></geometry>
-        <material name="silver"/>
-      </visual>
-      <collision>
-        <origin rpy="${pi/2.0} 0 0"/>
-        <geometry><cylinder radius="${wheel_radius}" length="${wheel_width}"/></geometry>
-      </collision>
-      <xacro:wheel_inertial mass="0.32" radius="${wheel_radius}" length="${wheel_width}"/>
-    </link>
-    <joint name="${prefix}_wheel_joint" type="continuous">
-      <parent link="base_link"/>
-      <child link="${prefix}_wheel_link"/>
-      <origin xyz="${x} ${y} 0"/>
-      <axis xyz="0 1 0"/>
-      <dynamics damping="0.02" friction="0.02"/>
-    </joint>
-  </xacro:macro>
-  <xacro:mecanum_wheel prefix="front_left"  x="${wheelbase/2.0}"  y="${track_width/2.0}"  roller_sign="1"/>
-  <xacro:mecanum_wheel prefix="front_right" x="${wheelbase/2.0}"  y="${-track_width/2.0}" roller_sign="-1"/>
-  <xacro:mecanum_wheel prefix="rear_left"   x="${-wheelbase/2.0}" y="${track_width/2.0}"  roller_sign="-1"/>
-  <xacro:mecanum_wheel prefix="rear_right"  x="${-wheelbase/2.0}" y="${-track_width/2.0}" roller_sign="1"/>
-  <xacro:macro name="motor" params="name x y">
-    <link name="${name}_motor_link">
-      <visual>
-        <origin rpy="${pi/2.0} 0 0"/>
-        <geometry><cylinder radius="0.018" length="0.045"/></geometry>
-        <material name="silver"/>
-      </visual>
-    </link>
-    <joint name="${name}_motor_joint" type="fixed">
-      <parent link="base_link"/>
-      <child link="${name}_motor_link"/>
-      <origin xyz="${x} ${y} 0.006"/>
-    </joint>
-  </xacro:macro>
-  <xacro:motor name="front_left"  x="${wheelbase/2.0}"  y="0.080"/>
-  <xacro:motor name="front_right" x="${wheelbase/2.0}"  y="-0.080"/>
-  <xacro:motor name="rear_left"   x="${-wheelbase/2.0}" y="0.080"/>
-  <xacro:motor name="rear_right"  x="${-wheelbase/2.0}" y="-0.080"/>
-  <link name="electronics_link">
-    <visual>
-      <geometry><box size="0.120 0.095 0.025"/></geometry>
-      <material name="blue"/>
-    </visual>
-  </link>
-  <joint name="electronics_joint" type="fixed">
-    <parent link="upper_plate_link"/>
-    <child link="electronics_link"/>
-    <origin xyz="-0.025 0 0.020"/>
-  </joint>
-  <link name="lidar_mount_link">
-    <visual>
-      <geometry><cylinder radius="0.035" length="0.055"/></geometry>
-      <material name="silver"/>
-    </visual>
-  </link>
-  <joint name="lidar_mount_joint" type="fixed">
-    <parent link="upper_plate_link"/>
-    <child link="lidar_mount_link"/>
-    <origin xyz="0.025 0 0.034"/>
-  </joint>
-  <link name="laser_link">
-    <visual>
-      <geometry><cylinder radius="0.043" length="0.030"/></geometry>
-      <material name="sensor_black"/>
-    </visual>
-  </link>
-  <joint name="laser_joint" type="fixed">
-    <parent link="lidar_mount_link"/>
-    <child link="laser_link"/>
-    <origin xyz="0 0 0.043"/>
-  </joint>
+  <joint name="base_footprint_joint" type="fixed"><parent link="base_footprint"/><child link="base_link"/><origin xyz="0 0 ${wheel_radius}"/></joint>
+  <link name="upper_plate_link"><visual><geometry><box size="${upper_length} ${upper_width} ${upper_height}"/></geometry><material name="black"/></visual><xacro:box_inertial mass="1.0" x="${upper_length}" y="${upper_width}" z="${upper_height}"/></link>
+  <joint name="upper_plate_joint" type="fixed"><parent link="base_link"/><child link="upper_plate_link"/><origin xyz="0 0 ${plate_gap}"/></joint>
+  <xacro:wheel name="front_left" x="${wheelbase/2.0}" y="${track_width/2.0}"/>
+  <xacro:wheel name="front_right" x="${wheelbase/2.0}" y="${-track_width/2.0}"/>
+  <xacro:wheel name="rear_left" x="${-wheelbase/2.0}" y="${track_width/2.0}"/>
+  <xacro:wheel name="rear_right" x="${-wheelbase/2.0}" y="${-track_width/2.0}"/>
+  <link name="lidar_mount_link"><visual><geometry><cylinder radius="0.035" length="0.055"/></geometry><material name="silver"/></visual></link>
+  <joint name="lidar_mount_joint" type="fixed"><parent link="upper_plate_link"/><child link="lidar_mount_link"/><origin xyz="0.025 0 0.034"/></joint>
+  <link name="laser_link"><visual><geometry><cylinder radius="0.043" length="0.030"/></geometry><material name="sensor_black"/></visual></link>
+  <joint name="laser_joint" type="fixed"><parent link="lidar_mount_link"/><child link="laser_link"/><origin xyz="0 0 0.043"/></joint>
   <link name="imu_link"/>
-  <joint name="imu_joint" type="fixed">
-    <parent link="base_link"/>
-    <child link="imu_link"/>
-    <origin xyz="0 0 0.025"/>
-  </joint>
+  <joint name="imu_joint" type="fixed"><parent link="base_link"/><child link="imu_link"/><origin xyz="0 0 0.025"/></joint>
   <link name="camera_link"/>
-  <joint name="camera_joint" type="fixed">
-    <parent link="upper_plate_link"/>
-    <child link="camera_link"/>
-    <origin xyz="${upper_length/2.0} 0 0.025"/>
-  </joint>
+  <joint name="camera_joint" type="fixed"><parent link="upper_plate_link"/><child link="camera_link"/><origin xyz="${upper_length/2.0} 0 0.025"/></joint>
 </robot>
